File: skymegaSMD.sch (KiCad schematic (older format))
At the start: 11 parts

Commit message: Finished basic schematic for the board.
Parts:
- removed C?: 1uF, ~, symbol C
- removed SERVO_? (x4): JP_3, symbol JP_3
- added BT1, I2C1: JP_4, symbol JP_4
- added C1, C2, C7: 0.1uF, ~, symbol C
- added C10: 100nF, symbol C
- added C12, C13, C14, C15, C16, C8, C9: 1uF, ~, symbol C
- added C3: 10uF, ~, symbol CP1
- added C4, C5: C, symbol C
- added C6: 10uF, tantalum, ~, symbol CP1
- added CP1, CP2: MOLEX-2, symbol MOLEX-2
- added D1, D2: RED, ~, symbol LED
- added D3, D4: BLUE, ~, symbol LED
- added D5: GREEN, ~, symbol LED
- added DOC1: I2C_DOC, symbol I2C_DOC
- added H1: HEAD3X2, symbol HEAD3X2
- added H_DOC1: ICSP_HEADER, symbol ICSP_HEADER
- added H_DOC2: H3X2-PINS-DOC, symbol H3X2-PINS-DOC
- added R1, R2, R3, R4, R7: 1K, ~, symbol R
- added R5, R6: R, ~, symbol R
- added R8: 10K, ~, symbol R
- added SERIAL1: M6, symbol JP_4
- added SERVO_5, SERVO_6, SERVO_7, SERVO_8: JP_3, symbol JP_3
- added SW1: SWITCH On_Off, symbol SWITCH_INV
- added SW2, SW3: SW_PUSH, ~, symbol SW_PUSH
- added U1: MIC5205, ~, symbol MIC5205
- added X1: 16Mhz, symbol CRYSTAL
- gave numbers to parts that had none: 6
Connections:
- net labels added: A6, A7, D11, D13, D2, D3, D4, D5, D6, D7, D8, DTR, MISO, MOSI, RESET, RX, SCK, SCL, SDA, SERVO_PWR_2, TX, VCC, Vin
- net labels removed: SERVO_PWR_0, SERVO_PWR_1
- wire segments 72 -> 197
- no-connect marks 0 -> 2
Other:
- note added: "5V-6V"
- note added: "ICSP"
- note added: "In Circuit Serial Programming header"
- note added: "Servo Connectors x8"
- note removed: "Servo Connectors x12"
- moved on the sheet: C11, IC1, SERVO_1, SERVO_2, SERVO_3, SERVO_4

Commit message: Footprint assignation and board layout.
Parts:
- removed DOC1: I2C_DOC, symbol I2C_DOC
- removed H_DOC1: ICSP_HEADER, symbol ICSP_HEADER
- removed H_DOC2: H3X2-PINS-DOC, symbol H3X2-PINS-DOC
- added K1: CONN_3, ~, symbol CONN_3
- added P1, P2: CONN_2, ~, symbol CONN_2
Connections:
- net labels added: D12
- wire segments 197 -> 204
Changed lines of the file:
@@
-EESchema Schematic File Version 2  date Tue 11 Mar 2014 23:06:10 CET
+EESchema Schematic File Version 2  date Wed 12 Mar 2014 14:01:58 CET
 LIBS:power
 LIBS:device
@@
 Sheet 1 1
 Title "Skymega-SMD"
-Date "11 mar 2014"
+Date "12 mar 2014"
 Rev "0.1"
 Comp "David Estévez Fernández"
@@
 	1    0    0    -1
 $EndComp
-$Comp
-L H3X2-PINS-DOC H_DOC2
-U 1 1 531F19A5
-P 10300 1700
-F 0 "H_DOC2" H 10650 1610 60  0001 C CNN
-F 1 "H3X2-PINS-DOC" H 10630 1510 60  0001 C CNN
-F 2 "" H 10300 1700 60  0001 C CNN
-F 3 "" H 10300 1700 60  0001 C CNN
-	1    10300 1700
-	1    0    0    -1
-$EndComp
-$Comp
-L ICSP_HEADER H_DOC1
-U 1 1 531F19AB
-P 10300 1200
-F 0 "H_DOC1" H 10650 1110 60  0001 C CNN
-F 1 "ICSP_HEADER" H 10630 1010 60  0001 C CNN
-F 2 "" H 10300 1200 60  0001 C CNN
-F 3 "" H 10300 1200 60  0001 C CNN
-	1    10300 1200
-	1    0    0    -1
-$EndComp
 Text Notes 8100 850  0    60   ~ 0
 In Circuit Serial Programming header
@@
 Text Label 4900 1450 2    60   ~ 0
 D10
-Text Label 4900 1550 2    60   ~ 0
+Text Label 4650 1550 2    60   ~ 0
 MOSI
-Text Label 4900 1650 2    60   ~ 0
+Text Label 4650 1650 2    60   ~ 0
 MISO
 Text Label 4650 1750 2    60   ~ 0
@@
 $EndComp
 $Comp
-L I2C_DOC DOC1
-U 1 1 531F809E
-P 3500 7500
-F 0 "DOC1" H 3650 7900 60  0001 C CNN
-F 1 "I2C_DOC" H 3650 7400 60  0001 C CNN
-F 2 "" H 3500 7500 60  0000 C CNN
-F 3 "" H 3500 7500 60  0000 C CNN
-	1    3500 7500
-	1    0    0    -1
-$EndComp
-$Comp
 L VCC #PWR014
 U 1 1 531F80AD
@@
 	1    0    0    -1
 $EndComp
+Connection ~ 9600 5500
+Connection ~ 8000 5450
+Text Label 4900 1550 2    60   ~ 0
+D11
+Text Label 4900 1650 2    60   ~ 0
+D12
+Wire Wire Line
+	6450 6200 6150 6200
+Wire Wire Line
+	6450 6300 6150 6300
+Wire Wire Line
+	6450 6400 6150 6400
+Text Label 6150 6200 0    60   ~ 0
+D5
+Text Label 6150 6300 0    60   ~ 0
+D6
+Text Label 6150 6400 0    60   ~ 0
+D7
+$Comp
+L CONN_2 P1
+U 1 1 53204DBE
+P 6800 5450
+F 0 "P1" V 6750 5450 40  0000 C CNN
+F 1 "CONN_2" V 6850 5450 40  0000 C CNN
+F 2 "~" H 6800 5450 60  0000 C CNN
+F 3 "~" H 6800 5450 60  0000 C CNN
+	1    6800 5450
+	1    0    0    -1
+$EndComp
+$Comp
+L CONN_2 P2
+U 1 1 53204DDF
+P 6800 5850
+F 0 "P2" V 6750 5850 40  0000 C CNN
+F 1 "CONN_2" V 6850 5850 40  0000 C CNN
+F 2 "~" H 6800 5850 60  0000 C CNN
+F 3 "~" H 6800 5850 60  0000 C CNN
+	1    6800 5850
+	1    0    0    -1
+$EndComp
+Wire Wire Line
+	6450 5350 6150 5350
+Wire Wire Line
+	6450 5550 6150 5550
+Text Label 6150 5350 0    60   ~ 0
+A6
+Text Label 6150 5550 0    60   ~ 0
+A7
+Wire Wire Line
+	6450 5750 6150 5750
+Wire Wire Line
+	6450 5950 6150 5950
+Text Label 6150 5750 0    60   ~ 0
+D3
+Text Label 6150 5950 0    60   ~ 0
+D4
+$Comp
+L CONN_3 K1
+U 1 1 53205012
+P 6800 6300
+F 0 "K1" V 6750 6300 50  0000 C CNN
+F 1 "CONN_3" V 6850 6300 40  0000 C CNN
+F 2 "~" H 6800 6300 60  0000 C CNN
+F 3 "~" H 6800 6300 60  0000 C CNN
+	1    6800 6300
+	1    0    0    -1
+$EndComp

Commit message: All components placed, capacitors bug solved.
Connections:
- wire segments 204 -> 245
Other:
- moved on the sheet: C11, C12, C13, C14, C15, C16, C8, C9

Commit message: More things routed.
Connections:
- wire segments 245 -> 200

Commit message: Version presented on thesis.
Connections:
- wire segments 200 -> 245
Other:
- note added: "5V LDO Regulator"
- note added: "Bluetooth\nconnector"
- note added: "Expansion headers"
- note added: "I2C bus connector"
- note added: "Microcontroller"
- note added: "Power connectors & LED indicators"
- note added: "Power\nflags"
- note added: "Reset push switch"
- note added: "Serial Port & LED indication"
- note added: "USER LED & USER Push switch"
- note removed: "ICSP"
- moved on the sheet: BT1, C1, C10, C11, C12, C13, C14, C15, C16, C2, C3, C4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
